File: electronics/MagicBox.kicad_sch (KiCad schematic)
At the start: 25 parts, among them SW1 SW_Push, SW2 SW_Push, SW3 SW_Push, SW4 SW_Push, SW5 SW_Push, SW6 SW_DPST_x2, SW7 RotaryEncoder_Switch, U1 ESP32-WROOM-32, U2 L7805

Commit message: first steps towards mk2.1 with new display
Parts:
- removed DS1: WC1602A, Display:WC1602A, symbol Display_Character:WC1602A
- removed R10, R6, R7, R8: 10k, symbol Device:R
- removed R3, R4, R5, R9: 1k, symbol Device:R
- removed SW4: SW_Push, symbol Switch:SW_Push
- added SW1_4: SW_Push, symbol Switch:SW_Push
- renumbered SW1 to SW1_1, SW2 to SW1_2, SW3 to SW1_3, SW6 to SW5, U1 to U1.U1, U2 to U1.U2
Connections:
- net +3.3V: now also SW1_4.1
- net SW_1: now also SW1_1.2
- net SW_2: now also SW1_2.2
- net SW_3: now also SW1_3.2
- new net SW_4: SW1_4.2
- no-connect marks 16 -> 17
Other:
- note added: "U1 - (ESP32 Node MCU)"
- note removed: "ESP32 - Node MCU"
- moved on the sheet: SW1_2, SW1_3

Commit message: small electronics and priting additions
Parts:
- added J1: Conn_01x05_Pin, symbol Connector:Conn_01x05_Pin
- added J2: Conn_01x05_Socket, symbol Connector:Conn_01x05_Socket
- added R3: 10k, symbol Device:R
Connections:
- net +3.3V: no longer SW7.C, SW7.S1
- net RE_CL: now also J2.1 (Pin_1); no longer SW7.B
- net RE_DT: now also J2.2 (Pin_2); no longer SW7.A
- net RE_SW: now also J2.3 (Pin_3); no longer R14.1
- net at R14.2, SW7.S2: now also R3.1
- new net: J1.5 (Pin_5), R3.2
- new net: J1.3 (Pin_3), R14.1
- new net: J1.1 (Pin_1), SW7.B
- new net: J1.2 (Pin_2), SW7.A
- new net: J1.4 (Pin_4), SW7.C, SW7.S1
Other:
- note added: "Rotary-Encoder-Module"

Commit message: starting overhawl of electronics
Other:
- note removed: "LCD - I2C"
Changed lines of the file:
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@@
-	)
-	(rectangle
-		(start 196.85 17.78)
-		(end 276.86 85.09)
-		(stroke
-			(width 0)
-			(type dash)
-		)
-		(fill
-			(type none)
-		)
 	)
 	(rectangle
@@
 		(effects
 			(font
-				(size 1.27 1.27)
-			)
-		)
-	)
-	(text "LCD - I2C"
-		(exclude_from_sim no)
-		(at 270.51 20.32 0)
-		(effects
-			(font
